File: cdf-alim-boost-24v-1.kicad_pcb (KiCad board)
At the start: 4 copper layers, 70 x 50 mm, 99 parts, among them J1 Conn_01x02, J2 Conn_01x02, J3 Conn_01x02, Q1 BSC019N04LS, Q2 BSC019N04LS, Q3 BSC019N04LS, Q4 BSC019N04LS, Q5 BSC019N04LS, U1 HT753-1, U2 TPS25983, U4 LM5122

Commit message: pcb(silk): add user text
Parts:
- added G***: LOGO, LOGO, F.Cu at (157.2, 82.0)
- added G***: LOGO, LOGO, B.Cu at (150.5, 75.5)
- added G*** (x3): LOGO, LOGO, B.Cu at (173.1, 78.3)
- added G***: LOGO, LOGO, B.Cu at (149.8, 94.5)
Other:
- board text added: "+"
- board text added: "+18V"
- board text added: "+24V"
- board text added: "+3V3"
- board text added: "+B"
- board text added: "-"
- board text added: "10A"
- board text added: "18V IN"
- board text added: "18V/10A INPUT"
- board text added: "24V OUT"
- board text added: "24V/10A OUTPUT"
- board text added: "CDF Alim Boost 24V 1"
- board text added: "EN"
- board text added: "JLCJLCJLCJLC"
- board text added: "Rev 01"
- board text added: "Rémi Ait-Younes 26-10"
- board text added: "edition"
- board text added: "アイドルライフメガパック"
